File: KiCad/Automatic AC Line Voltage Selector TL431/Automatic AC Line Voltage Selector TL431.kicad_sch (KiCad schematic)
At the start: 38 parts, among them J1 AC Line, J2 Conn_01x03, J3 Conn_01x03, K1 G5LE-1, K2 G5LE-1, Q1 BC817, Q2 STD3NM60, U1 TL431D

Commit message: Update
Other:
- company: (none) -> RTEK1000
- title: (none) -> Automatic AC voltage selector
Changed lines of the file:
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@@
 (kicad_sch (version 20230121) (generator eeschema)
   (paper "A4")
+  (title_block
+    (title "Automatic AC voltage selector")
+    (date "2023-07-09")
+    (rev "1.0")
+    (company "RTEK1000")
+  )
   (junction (at 91.948 137.668) (diameter 0) (color 0 0 0 0)
   )

Commit message: Update
Parts:
- F1: value Fuse -> T0.5AH
Changed lines of the file:
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@@
   (symbol (lib_id "Device:Fuse") (at 65.786 71.374 90) (unit 1)
     (in_bom yes) (on_board yes) (dnp no) (fields_autoplaced)
-    (property "Reference" "F1" (at 65.786 66.548 90)
+    (property "Reference" "F1" (at 65.786 67.31 90)
       (effects (font (size 1.27 1.27)))
     )
-    (property "Value" "Fuse" (at 65.786 69.088 90)
+    (property "Value" "T0.5AH" (at 65.786 69.85 90)
       (effects (font (size 1.27 1.27)))
     )

Commit message: Update
Parts:
- RV1: value 271 -> 431
Changed lines of the file:
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@@
       (effects (font (size 1.27 1.27)) (justify right))
     )
-    (property "Value" "271" (at 67.818 85.1177 0)
+    (property "Value" "431" (at 67.818 85.1177 0)
       (effects (font (size 1.27 1.27)) (justify right))
     )
@@
   )
   (symbol (lib_id "Device:Fuse") (at 65.786 71.374 90) (unit 1)
-    (in_bom yes) (on_board yes) (dnp no) (fields_autoplaced)
-    (property "Reference" "F1" (at 65.786 67.31 90)
-      (effects (font (size 1.27 1.27)))
-    )
-    (property "Value" "T0.5AH" (at 65.786 69.85 90)
-      (effects (font (size 1.27 1.27)))
-    )
+    (in_bom yes) (on_board yes) (dnp no)
+    (property "Reference" "F1" (at 66.04 66.675 90)
+      (effects (font (size 1.27 1.27)))
+    )
+    (property "Value" "T0.5AH" (at 66.04 69.215 90)
+      (effects (font (size 1.27 1.27)))
+    )
